File: citrus-board/citrus-board.kicad_sch (KiCad schematic)
At the start: 63 parts, among them J1 SHOU_HAN_USB_C_Receptacle_USB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, J2 Conn_01x03_MountingPin, J3 Conn_01x02, J5 0.5mm FPC, J6 Conn_01x13, J7 Conn_01x13, SW1 SW_Push, SW2 SW_Push, U1 W25Q128JVS, U2 BQ24074RGT, U3 TPS63000-Q1, U4 RP2354A, Y1 Crystal_GND24

Commit message: finish routing
Parts:
- removed C16, C17, C18, C19: 100n, Capacitor_SMD:C_0402_1005Metric, symbol Device:C_Small
- added H1, H2, H3, H4: MountingHole, MountingHole:MountingHole_2.1mm, symbol Mechanical:MountingHole
- C4: renamed from C1; footprint Capacitor_SMD:C_0402_1005Metric -> Capacitor_SMD:C_0805_2012Metric
- D2: value GREEN -> RED; footprint LED_SMD:LED_0805_2012Metric -> LED_SMD:LED_0603_1608Metric; LCSC Part # C2297 -> C2286
- J1: symbol Connector:USB_C_Receptacle_USB2.0_16P -> symbols:SHOU_HAN_USB_C_Receptacle_USB2.0_16P
- J4: renamed from J5; symbol Connector:Conn_01x22_Pin -> Connector_Generic_Shielded:Conn_01x22_Shielded
- J5: renamed from J6; footprint Connector_PinHeader_2.54mm:PinHeader_1x13_P2.54mm_Vertical -> Connector_PinHeader_2.54mm:PinHeader_1x14_P2.54mm_Vertical; symbol Connector_Generic:Conn_01x13 -> Connector_Generic:Conn_01x14
- J6: renamed from J7; footprint Connector_PinHeader_2.54mm:PinHeader_1x13_P2.54mm_Vertical -> Connector_PinHeader_2.54mm:PinHeader_1x14_P2.54mm_Vertical; symbol Connector_Generic:Conn_01x13 -> Connector_Generic:Conn_01x14
- L2: renamed from L1; value 3.3u -> 3.3uH
- R1: renamed from R11; footprint Resistor_SMD:R_01005_0402Metric -> Resistor_SMD:R_0402_1005Metric
- R11: renamed from R3; value 33 -> 33R
- R12: renamed from R17; footprint Resistor_SMD:R_01005_0402Metric -> Resistor_SMD:R_0402_1005Metric
- R13: renamed from R4; value 27 -> 27R
- R14: renamed from R5; value 27 -> 27R
- R15: renamed from R9; footprint Resistor_SMD:R_01005_0402Metric -> Resistor_SMD:R_0402_1005Metric
- R17: renamed from R8; footprint Resistor_SMD:R_01005_0402Metric -> Resistor_SMD:R_0402_1005Metric
- R2: renamed from R14; footprint Resistor_SMD:R_01005_0402Metric -> Resistor_SMD:R_0402_1005Metric
- R3: renamed from R10; footprint Resistor_SMD:R_01005_0402Metric -> Resistor_SMD:R_0402_1005Metric
- R6: renamed from R12; footprint Resistor_SMD:R_01005_0402Metric -> Resistor_SMD:R_0402_1005Metric
- R7: renamed from R13; footprint Resistor_SMD:R_01005_0402Metric -> Resistor_SMD:R_0402_1005Metric
- R8: renamed from R15; footprint Resistor_SMD:R_01005_0402Metric -> Resistor_SMD:R_0402_1005Metric
- R9: renamed from R16; footprint Resistor_SMD:R_01005_0402Metric -> Resistor_SMD:R_0402_1005Metric
- U2: renamed from U3; LCSC Part # (none) -> C28060
- renumbered C21 to C1, C4 to C10, C5 to C11, C6 to C12, C7 to C13, C8 to C14, C26 to C15, C28 to C16, C9 to C17, C10 to C18, C11 to C19, C22 to C2, C12 to C20, C13 to C21, C14 to C22, C15 to C23, C20 to C27, C25 to C3, C23 to C5, C24 to C6, C2 to C7, C27 to C8, C3 to C9, J3 to J2, J2 to J3, L2 to L1, R6 to R10, R7 to R16, R1 to R4, R2 to R5, U2 to U1, U4 to U3, U1 to U4
Connections:
- net GPIO28 is gone; now on net GPIO28//SDA: U3.42 (GPIO28_ADC2)
- net GPIO29 is gone; now on net GPIO29//SCL: U3.43 (GPIO29_ADC3)
- net +3V3: now also J4.22 (Pin_22), J6.10 (Pin_10), J6.8 (Pin_8); no longer J4.1 (Pin_1), J6.9 (Pin_9)
- net D+: now also J1.A6 (D+), J1.B6 (D+); no longer J1.A7 (D-), J1.B7 (D-)
- net D-: now also J1.A7 (D-), J1.B7 (D-); no longer J1.A6 (D+), J1.B6 (D+)
- net EN: now also J6.11 (Pin_11); no longer J6.10 (Pin_10)
- net GND: now also J1.13 (EH), J1.14 (EH), J1.A1B12 (GND), J1.B1A12 (GND), J4.1 (Pin_1), J4.23 (Shield), J4.24 (Shield), J6.6 (Pin_6); no longer C6.1, C7.1, J1.A1 (GND), J1.A12 (GND), J1.B1 (GND), J1.B12 (GND), J4.22 (Pin_22), J6.11 (Pin_11), J6.5 (Pin_5), R7.1, R8.1, R9.1, U1.10 (OUT), U1.11 (OUT), U1.5 (EN2), U2.5 (VIN)
- net GPIO10: now also J4.18 (Pin_18); no longer J4.5 (Pin_5)
- net GPIO11: now also J4.17 (Pin_17); no longer J4.6 (Pin_6)
- net GPIO12: now also J4.12 (Pin_12); no longer J4.11 (Pin_11)
- net GPIO13: now also J4.11 (Pin_11); no longer J4.12 (Pin_12)
- net GPIO14: now also J4.9 (Pin_9); no longer J4.14 (Pin_14)
- net GPIO15: now also J4.8 (Pin_8); no longer J4.15 (Pin_15)
- net GPIO16: now also J4.6 (Pin_6); no longer J4.17 (Pin_17)
- net GPIO17: now also J4.5 (Pin_5); no longer J4.18 (Pin_18)
- net GPIO18: now also J4.3 (Pin_3); no longer J4.20 (Pin_20)
- net GPIO19: now also J4.2 (Pin_2); no longer J4.21 (Pin_21)
- net GPIO21: now also J5.14 (Pin_14); no longer J6.1 (Pin_1)
- net GPIO22: now also J6.1 (Pin_1); no longer J6.2 (Pin_2)
- net GPIO23: now also J6.2 (Pin_2); no longer J6.3 (Pin_3)
- net GPIO24: now also J6.3 (Pin_3); no longer J6.4 (Pin_4)
- net GPIO25: now also J6.4 (Pin_4); no longer J6.6 (Pin_6)
- net GPIO26: now also J6.5 (Pin_5); no longer J6.8 (Pin_8)
- net GPIO28//SDA: now also J4.21 (Pin_21); no longer J4.2 (Pin_2)
- net GPIO29//SCL: now also J4.20 (Pin_20); no longer J4.3 (Pin_3)
- net VBUS: now also J1.A4B9 (VBUS), J1.B4A9 (VBUS), J6.14 (Pin_14); no longer J1.A4 (VBUS), J1.A9 (VBUS), J1.B4 (VBUS), J1.B9 (VBUS), J6.13 (Pin_13)
- net RUN: now reaches R12.2, SW2.2, U3.26 (RUN)
- net RUN: now also J6.9 (Pin_9)
- net U3-USB_DP: now reaches R13.2, U3.52 (USB_DP)
- net U3-USB_DN: now reaches R14.2, U3.51 (USB_DM)
- new net BC_OUT: C6.1, C7.1, J6.13 (Pin_13), R7.1, R8.1, R9.1, U1.10 (OUT), U1.11 (OUT), U1.5 (EN2), U2.5 (VIN)
Other:
- moved on the sheet: C6, D1, R7

Commit message: update fields + production export
Parts:
- C1, C2: LCSC Part # (none) -> C1548
- C10, C12, C14, C5, C6, C9: LCSC Part # (none) -> C23733
- C11, C13, C17, C18, C19, C20, C21, C22, C23, C27, C8: LCSC Part # (none) -> C307331
- C15, C16, C7: footprint Capacitor_SMD:C_0402_1005Metric -> Capacitor_SMD:C_0805_2012Metric; LCSC Part # (none) -> C1713
- C3: footprint Capacitor_SMD:C_0402_1005Metric -> Capacitor_SMD:C_0603_1608Metric; LCSC Part # (none) -> C1592
- C4: LCSC Part # (none) -> C1713
- J1: LCSC Part # (none) -> C2765186
- J5, J6: now left out of the parts list
- L2: LCSC Part # (none) -> C42411119
- R1, R10: LCSC Part # (none) -> C270651
- R11: LCSC Part # (none) -> C25105
- R12, R15, R17, R6: LCSC Part # (none) -> C25744
- R13, R14: LCSC Part # (none) -> C25100
- R16: LCSC Part # (none) -> C17477
- R2: LCSC Part # (none) -> C67014
- R3: LCSC Part # (none) -> C227387
- R4, R5: LCSC Part # (none) -> C25905
- R7: LCSC Part # (none) -> C25867
- R8: LCSC Part # (none) -> C25076
- R9: LCSC Part # (none) -> C25741
- U3: LCSC Part # (none) -> C41378174
- U4: LCSC Part # (none) -> C97521
- Y1: LCSC Part # (none) -> C20625731
