File: pcb/citrus-board.kicad_sch (KiCad schematic)
At the start: 63 parts, among them J1 SHOU_HAN_USB_C_Receptacle_USB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, J2 Conn_01x02, J3 Conn_01x03_MountingPin, J4 0.5mm FPC, J5 Conn_01x13, J6 Conn_01x13, SW1 SW_Push, SW2 SW_Push, U1 BQ24074RGT, U2 TPS63000-Q1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

Commit message: castellated holes + better silkscreen + new images
Parts:
- J5, J6: footprint Connector_PinHeader_2.54mm:PinHeader_1x14_P2.54mm_Vertical -> citrus-lib:Conn_01x14_Castellated
Changed lines of the file:
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@@
 			)
 		)
-		(property "Footprint" "Connector_PinHeader_2.54mm:PinHeader_1x14_P2.54mm_Vertical"
+		(property "Footprint" "citrus-lib:Conn_01x14_Castellated"
 			(at 360.68 142.24 0)
 			(hide yes)
@@
 			)
 		)
-		(property "Footprint" "Connector_PinHeader_2.54mm:PinHeader_1x14_P2.54mm_Vertical"
+		(property "Footprint" "citrus-lib:Conn_01x14_Castellated"
 			(at 363.22 144.78 0)
 			(hide yes)
